File: CurrentServo.sch (KiCad schematic (older format))
At the start: 32 parts, among them P1 POWER, P2 SENSE, P3 V_DAC, P4 VREF, P5 HH_IN, P6 OUT, U1 VHP4Z, U2 INA105, U3 78L05, U4 INA105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

Commit message: Files sent for manufacture
Parts:
- U6: footprint Opto-Devices:Optocoupler_6pin_wide_Stile-I -> local:TLP116A
Changed lines of the file:
@@
 EESchema Schematic File Version 2
-LIBS:CurrentServo-rescue
 LIBS:CurrentServo
 LIBS:power
@@
 Sheet 1 3
 Title "Helmholtz Current Servo"
-Date ""
+Date "2016-11-14"
 Rev ""
 Comp "Kjaergaard Lab"
@@
 F 0 "U6" H 8950 1750 50  0000 L CNN
 F 1 "TLP116A" H 9150 1750 50  0000 L CNN
-F 2 "Opto-Devices:Optocoupler_6pin_wide_Stile-I" H 8950 1350 50  0001 L CIN
+F 2 "local:TLP116A" H 8950 1350 50  0001 L CIN
 F 3 "" H 9150 1550 50  0000 L CNN
 	1    9150 1550
